File: hardware/cpx-module1-F.sch (EAGLE design)
At the start: 6 parts, among them T1 TOUCHPADROUND1, T2 TOUCHPADROUND1, T3 TOUCHPADROUND1, T4 TOUCHPADROUND1, U1 CIRCUITPLAYGROUNDEXPRESS

Commit message: added protection diodes and filter caps, added pdfs
Parts:
- removed T3: TOUCHPADROUND1, todstuff:TOUCHPADROUND1
Connections:
- net A1: now also T2.TOUCH
- net A4: no longer T3.TOUCH
- net A5: no longer T2.TOUCH
Changed lines of the file:
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@@
 <part name="T1" library="todstuff" library_urn="urn:adsk.eagle:library:1731349" deviceset="TOUCHPAD" device="" technology="ROUND1"/>
 <part name="T2" library="todstuff" library_urn="urn:adsk.eagle:library:1731349" deviceset="TOUCHPAD" device="" technology="ROUND1"/>
-<part name="T3" library="todstuff" library_urn="urn:adsk.eagle:library:1731349" deviceset="TOUCHPAD" device="" technology="ROUND1"/>
 <part name="J10" library="SparkFun-Connectors" library_urn="urn:adsk.eagle:library:513" deviceset="CONN_10" device="&quot;" package3d_urn="urn:adsk.eagle:package:38157/1"/>
 <part name="GND18" library="supply1" library_urn="urn:adsk.eagle:library:371" deviceset="GND" device=""/>
@@
 <instance part="T1" gate="G$1" x="40.64" y="111.76" rot="R180"/>
 <instance part="T2" gate="G$1" x="40.64" y="124.46" rot="R180"/>
-<instance part="T3" gate="G$1" x="40.64" y="137.16" rot="R180"/>
 <instance part="J10" gate="G$1" x="99.06" y="127" rot="R270"/>
 <instance part="GND18" gate="1" x="91.44" y="99.06"/>
@@
 </segment>
 <segment>
-<pinref part="T3" gate="G$1" pin="TOUCH"/>
-<wire x1="50.8" y1="137.16" x2="60.96" y2="137.16" width="0.1524" layer="91"/>
-<label x="58.42" y="137.16" size="1.778" layer="95"/>
-</segment>
-<segment>
 <pinref part="J10" gate="G$1" pin="3"/>
 <wire x1="86.36" y1="116.84" x2="86.36" y2="109.22" width="0.1524" layer="91"/>
@@
 <wire x1="40.64" y1="73.66" x2="27.94" y2="73.66" width="0.1524" layer="91"/>
 <label x="27.94" y="73.66" size="1.778" layer="95"/>
-</segment>
-<segment>
-<pinref part="T2" gate="G$1" pin="TOUCH"/>
-<wire x1="50.8" y1="124.46" x2="60.96" y2="124.46" width="0.1524" layer="91"/>
-<label x="58.42" y="124.46" size="1.778" layer="95"/>
 </segment>
 <segment>
@@
 <label x="104.14" y="109.22" size="1.778" layer="95" rot="R90"/>
 </segment>
+<segment>
+<pinref part="T2" gate="G$1" pin="TOUCH"/>
+<wire x1="50.8" y1="124.46" x2="60.96" y2="124.46" width="0.1524" layer="91"/>
+<label x="58.42" y="124.46" size="1.778" layer="95"/>
+</segment>
 </net>
